Commit message: Get combined Sawyer/Robotiq working in Gazebo

File: urdf/sawyer_combined.urdf.xacro (robot description, xacro)
@@ -1,11 +1,17 @@
 <?xml version="1.0" ?>
-<robot name="sawyer_robotiq" xmlns:xacro="http://www.ros.org/wiki/xacro">
-<!--  <xacro:include filename="$(find sawyer_description)/urdf/sawyer.urdf.xacro">
+<robot name="sawyer" xmlns:xacro="http://www.ros.org/wiki/xacro">
+  <xacro:arg name="gazebo" default="true"/>
+  <xacro:arg name="pedestal" default="true"/>
+  <xacro:arg name="static" default="true"/>
+  <xacro:arg name="electric_gripper" default="false"/>
+  <xacro:include filename="$(find sawyer_description)/urdf/sawyer.urdf.xacro">
+    <xacro:arg name="gazebo" value="${gazebo}"/>
+    <xacro:arg name="pedestal" value="${pedestal}"/>
+    <xacro:arg name="static" value="${static}"/>
+    <xacro:arg name="electric_gripper" value="${electric_gripper}"/>
   </xacro:include>
--->
   <xacro:include filename="$(find robotiq_2f_85_gripper_visualization)/urdf/robotiq_arg2f_85_model.xacro">
   </xacro:include>
-<!--
-  <joint name="robotiq_gripper_base_joint" type="fixed" >
+  <joint name="right_gripper_base_joint" type="fixed" >
         <origin xyz="0.0 0.0 0.001" rpy="0.0 0.0 1.5707"/>
         <parent link="right_hand" />
@@ -14,8 +20,25 @@
     <link name="right_gripper_base"/>
     <joint name="robotiq_c_model_adapter" type="fixed" >
-        <origin xyz="0.0 0.0 0.09712" rpy="0.0 0.0 0.0"/>
+        <origin xyz="0.0 0.0 0.00" rpy="0.0 0.0 0.0"/>
         <parent link="right_gripper_base" />
         <child link="robotiq_arg2f_base_link" />
     </joint>
--->
+    <joint name="right_gripper_tip_joint" type="fixed">
+      <origin rpy="0 0 0" xyz="0 0 0.1268"/>
+      <parent link="robotiq_arg2f_base_link"/>
+      <child link="right_gripper_tip"/>
+    </joint>
+    <!-- Electric Gripper Tip link -->
+    <link name="right_gripper_tip">
+      <inertial>
+        <origin xyz="0 0 0" rpy="0 0 0"/>
+        <mass value="2e-06"/>
+        <inertia ixx="1.1e-09" ixy="0" ixz="0" iyy="1.1e-09" iyz="0" izz="1.1e-09"/>
+      </inertial>
+    </link>
+  <link name="world"/>
+  <joint name="fixed" type="fixed">
+      <parent link="world"/>
+      <child link="base"/>
+  </joint>
 </robot>

Commit message: Meshes and collision objects updated

File: urdf/sawyer_combined.urdf.xacro (robot description, xacro)
@@ -1,17 +1,11 @@
 <?xml version="1.0" ?>
-<robot name="sawyer" xmlns:xacro="http://www.ros.org/wiki/xacro">
-  <xacro:arg name="gazebo" default="true"/>
-  <xacro:arg name="pedestal" default="true"/>
-  <xacro:arg name="static" default="true"/>
-  <xacro:arg name="electric_gripper" default="false"/>
-  <xacro:include filename="$(find sawyer_description)/urdf/sawyer.urdf.xacro">
-    <xacro:arg name="gazebo" value="${gazebo}"/>
-    <xacro:arg name="pedestal" value="${pedestal}"/>
-    <xacro:arg name="static" value="${static}"/>
-    <xacro:arg name="electric_gripper" value="${electric_gripper}"/>
+<robot name="sawyer_robotiq" xmlns:xacro="http://www.ros.org/wiki/xacro">
+<!--  <xacro:include filename="$(find sawyer_description)/urdf/sawyer.urdf.xacro">
   </xacro:include>
+-->
   <xacro:include filename="$(find robotiq_2f_85_gripper_visualization)/urdf/robotiq_arg2f_85_model.xacro">
   </xacro:include>
-  <joint name="right_gripper_base_joint" type="fixed" >
+<!--
+  <joint name="robotiq_gripper_base_joint" type="fixed" >
         <origin xyz="0.0 0.0 0.001" rpy="0.0 0.0 1.5707"/>
         <parent link="right_hand" />
@@ -20,25 +14,8 @@
     <link name="right_gripper_base"/>
     <joint name="robotiq_c_model_adapter" type="fixed" >
-        <origin xyz="0.0 0.0 0.00" rpy="0.0 0.0 0.0"/>
+        <origin xyz="0.0 0.0 0.09712" rpy="0.0 0.0 0.0"/>
         <parent link="right_gripper_base" />
         <child link="robotiq_arg2f_base_link" />
     </joint>
-    <joint name="right_gripper_tip_joint" type="fixed">
-      <origin rpy="0 0 0" xyz="0 0 0.1268"/>
-      <parent link="robotiq_arg2f_base_link"/>
-      <child link="right_gripper_tip"/>
-    </joint>
-    <!-- Electric Gripper Tip link -->
-    <link name="right_gripper_tip">
-      <inertial>
-        <origin xyz="0 0 0" rpy="0 0 0"/>
-        <mass value="2e-06"/>
-        <inertia ixx="1.1e-09" ixy="0" ixz="0" iyy="1.1e-09" iyz="0" izz="1.1e-09"/>
-      </inertial>
-    </link>
-  <link name="world"/>
-  <joint name="fixed" type="fixed">
-      <parent link="world"/>
-      <child link="base"/>
-  </joint>
+-->
 </robot>

Commit message: sawyer_world.launch added

File: urdf/sawyer_combined.urdf.xacro (robot description, xacro)
@@ -13,4 +13,5 @@
   <xacro:include filename="$(find robotiq_2f_85_gripper_visualization)/urdf/robotiq_arg2f_85_model.xacro">
   </xacro:include>
+  <link name="world"/>
   <joint name="right_gripper_base_joint" type="fixed" >
         <origin xyz="0.0 0.0 0.001" rpy="0.0 0.0 1.5707"/>
@@ -37,5 +38,4 @@
       </inertial>
     </link>
-  <link name="world"/>
   <joint name="fixed" type="fixed">
       <parent link="world"/>
