Commit message: Except room urdf, all other problems cleaned

File: urdf/conveyor.urdf.xacro (robot description, xacro)
@@ -512,8 +512,8 @@
     </inertial>
     </link>
-  <joint name="frame_to_belt" type="revolute">
+  <joint name="frame_to_belt" type="fixed">
     <origin rpy="0 0 0" xyz="0.75 0 0.73" />
-    <axis xyz="1 0 0" />
-    <limit lower="0.0" upper="6.28319" effort="1000.0" velocity="0.5"/>
+    <!--axis xyz="1 0 0" />
+    <limit lower="0.0" upper="6.28319" effort="1000.0" velocity="0.5"/-->
     <parent link="frame"/>
     <child link="belt"/>
@@ -541,5 +541,5 @@
     </inertial>
     </link>
-   <transmission name="tran1">
+   <!--transmission name="tran1">
 	<type>transmission_interface/SimpleTransmission</type>
 	<joint name="frame_to_roller1">
@@ -701,4 +701,10 @@
 	</actuator>
    </transmission>
+    <gazebo>
+	<static>false</static>
+	<plugin name="gazebo_ros_control" filename="libgazebo_ros_control.so">
+	</plugin>
+	<robotNamespace>conveyor_table</robotNamespace>
+    </gazebo-->
     <gazebo reference="frame">
         <material>Gazebo/Grey</material>
@@ -707,9 +713,3 @@
         <material>Gazebo/FlatBlack</material>
     </gazebo>
-    <gazebo>
-	<static>false</static>
-	<plugin name="gazebo_ros_control" filename="libgazebo_ros_control.so">
-	</plugin>
-	<!--robotNamespace>conveyor_table</robotNamespace-->
-    </gazebo>
 </robot>

Commit message: Includes Saurabh's changes - cleaned up

File: urdf/conveyor.urdf.xacro (robot description, xacro)
@@ -1,5 +1,16 @@
 <?xml version="1.0"?>
 <robot name="conveyor_table" xmlns:xacro="http://www.ros.org/wiki/xacro">
+<!-- Author: Prasanth Suresh (ps32611@uga.edu); Description: Conveyor table to be used by Sawyer -->
+<!-- Do not edit/replicate without permission -->
+<!--
+Belt Width:15.7inch ;
+Belt Thickness:0.07inch ;
+Conveyor Length:59inch
+Conveyor High:29.5inch
+-->
   <xacro:arg name="gazebo" default="false"/>
+  <xacro:arg name="load_rollers" default="false"/>
+  <xacro:arg name="load_motors" default="false"/>
+  <xacro:arg name="load_railings" default="true"/>
   <material name="white">
     <color rgba="1 1 1 1"/>
@@ -24,7 +35,7 @@
     <parent link="world"/>
     <child link="frame"/>
-<xacro:if value="$(arg gazebo)">
-    <dynamics damping="10.0" friction="5.0"/>
-</xacro:if>
+   <xacro:if value="$(arg gazebo)">
+    <dynamics damping="10.0" friction="5.0"/>
+   </xacro:if>
   </joint>
     <link name="frame" type="fixed" >
@@ -34,5 +45,4 @@
 		<mesh filename="package://sawyer_irl_project/meshes/frame.stl"/>
 	  </geometry>
-	<!--<material name="sawyer_red"/>-->
        </visual>
 	<collision>
@@ -48,4 +58,5 @@
       </inertial>
     </link>
+<xacro:if value="$(arg load_rollers)">
   <joint name="frame_to_roller1" type="revolute">
     <origin xyz="0.75 -0.7 0.73" rpy="0 0 0"/>
@@ -54,9 +65,9 @@
     <parent link="frame"/>
     <child link="roller1"/>
-<xacro:if value="$(arg gazebo)">
-    <dynamics damping="10.0" friction="5.0"/>
-</xacro:if>
-   </joint>
-   <link name="roller1" type="fixed" > <!-- Every roller is 0.1 from previous center -->
+   <xacro:if value="$(arg gazebo)">
+    <dynamics damping="10.0" friction="5.0"/>
+   </xacro:if>
+   </joint>
+   <link name="roller1" type="fixed" >
        <visual>
 	<origin rpy="0 0 0" xyz="0 0 0" />
@@ -83,9 +94,9 @@
     <parent link="frame"/>
     <child link="roller2"/>
-<xacro:if value="$(arg gazebo)">
-    <dynamics damping="10.0" friction="5.0"/>
-</xacro:if>
-   </joint>
-   <link name="roller2" type="fixed" > <!-- Every roller is 0.1 from previous center -->
+   <xacro:if value="$(arg gazebo)">
+    <dynamics damping="10.0" friction="5.0"/>
+   </xacro:if>
+   </joint>
+   <link name="roller2" type="fixed" >
        <visual>
 	<origin rpy="0 0 0" xyz="0 0 0" />
@@ -112,9 +123,9 @@
     <parent link="frame"/>
     <child link="roller3"/>
-<xacro:if value="$(arg gazebo)">
-    <dynamics damping="10.0" friction="5.0"/>
-</xacro:if>
-   </joint>
-   <link name="roller3" type="fixed" > <!-- Every roller is 0.1 from previous center -->
+   <xacro:if value="$(arg gazebo)">
+    <dynamics damping="10.0" friction="5.0"/>
+   </xacro:if>
+   </joint>
+   <link name="roller3" type="fixed" >
        <visual>
 	<origin rpy="0 0 0" xyz="0 0 0" />
@@ -141,9 +152,9 @@
     <parent link="frame"/>
     <child link="roller4"/>
-<xacro:if value="$(arg gazebo)">
-    <dynamics damping="10.0" friction="5.0"/>
-</xacro:if>
-   </joint>
-   <link name="roller4" type="fixed" > <!-- Every roller is 0.1 from previous center -->
+   <xacro:if value="$(arg gazebo)">
+    <dynamics damping="10.0" friction="5.0"/>
+   </xacro:if>
+   </joint>
+   <link name="roller4" type="fixed" >
        <visual>
 	<origin rpy="0 0 0" xyz="0 0 0" />
@@ -170,9 +181,9 @@
     <parent link="frame"/>
     <child link="roller5"/>
-<xacro:if value="$(arg gazebo)">
-    <dynamics damping="10.0" friction="5.0"/>
-</xacro:if>
-   </joint>
-   <link name="roller5" type="fixed" > <!-- Every roller is 0.1 from previous center -->
+   <xacro:if value="$(arg gazebo)">
+    <dynamics damping="10.0" friction="5.0"/>
+   </xacro:if>
+   </joint>
+   <link name="roller5" type="fixed" >
        <visual>
 	<origin rpy="0 0 0" xyz="0 0 0" />
@@ -199,9 +210,9 @@
     <parent link="frame"/>
     <child link="roller6"/>
-<xacro:if value="$(arg gazebo)">
-    <dynamics damping="10.0" friction="5.0"/>
-</xacro:if>
-   </joint>
-   <link name="roller6" type="fixed" > <!-- Every roller is 0.1 from previous center -->
+   <xacro:if value="$(arg gazebo)">
+    <dynamics damping="10.0" friction="5.0"/>
+   </xacro:if>
+   </joint>
+   <link name="roller6" type="fixed" >
        <visual>
 	<origin rpy="0 0 0" xyz="0 0 0" />
@@ -228,9 +239,9 @@
     <parent link="frame"/>
     <child link="roller7"/>
-<xacro:if value="$(arg gazebo)">
-    <dynamics damping="10.0" friction="5.0"/>
-</xacro:if>
-   </joint>
-   <link name="roller7" type="fixed" > <!-- Every roller is 0.1 from previous center -->
+   <xacro:if value="$(arg gazebo)">
+    <dynamics damping="10.0" friction="5.0"/>
+   </xacro:if>
+   </joint>
+   <link name="roller7" type="fixed" >
        <visual>
 	<origin rpy="0 0 0" xyz="0 0 0" />
@@ -257,9 +268,9 @@
     <parent link="frame"/>
     <child link="roller8"/>
-<xacro:if value="$(arg gazebo)">
-    <dynamics damping="10.0" friction="5.0"/>
-</xacro:if>
-   </joint>
-   <link name="roller8" type="fixed" > <!-- Every roller is 0.1 from previous center -->
+   <xacro:if value="$(arg gazebo)">
+    <dynamics damping="10.0" friction="5.0"/>
+   </xacro:if>
+   </joint>
+   <link name="roller8" type="fixed" >
        <visual>
 	<origin rpy="0 0 0" xyz="0 0 0" />
@@ -286,9 +297,9 @@
     <parent link="frame"/>
     <child link="roller9"/>
-<xacro:if value="$(arg gazebo)">
-    <dynamics damping="10.0" friction="5.0"/>
-</xacro:if>
-   </joint>
-   <link name="roller9" type="fixed" > <!-- Every roller is 0.1 from previous center -->
+   <xacro:if value="$(arg gazebo)">
+    <dynamics damping="10.0" friction="5.0"/>
+   </xacro:if>
+   </joint>
+   <link name="roller9" type="fixed" >
        <visual>
 	<origin rpy="0 0 0" xyz="0 0 0" />
@@ -315,9 +326,9 @@
     <parent link="frame"/>
     <child link="roller10"/>
-<xacro:if value="$(arg gazebo)">
-    <dynamics damping="10.0" friction="5.0"/>
-</xacro:if>
-   </joint>
-   <link name="roller10" type="fixed" > <!-- Every roller is 0.1 from previous center -->
+   <xacro:if value="$(arg gazebo)">
+    <dynamics damping="10.0" friction="5.0"/>
+   </xacro:if>
+   </joint>
+   <link name="roller10" type="fixed" >
        <visual>
 	<origin rpy="0 0 0" xyz="0 0 0" />
@@ -344,9 +355,9 @@
     <parent link="frame"/>
     <child link="roller11"/>
-<xacro:if value="$(arg gazebo)">
-    <dynamics damping="10.0" friction="5.0"/>
-</xacro:if>
-   </joint>
-   <link name="roller11" type="fixed" > <!-- Every roller is 0.1 from previous center -->
+   <xacro:if value="$(arg gazebo)">
+    <dynamics damping="10.0" friction="5.0"/>
+   </xacro:if>
+   </joint>
+   <link name="roller11" type="fixed" >
        <visual>
 	<origin rpy="0 0 0" xyz="0 0 0" />
@@ -373,9 +384,9 @@
     <parent link="frame"/>
     <child link="roller12"/>
-<xacro:if value="$(arg gazebo)">
-    <dynamics damping="10.0" friction="5.0"/>
-</xacro:if>
-   </joint>
-   <link name="roller12" type="fixed" > <!-- Every roller is 0.1 from previous center -->
+   <xacro:if value="$(arg gazebo)">
+    <dynamics damping="10.0" friction="5.0"/>
+   </xacro:if>
+   </joint>
+   <link name="roller12" type="fixed" >
        <visual>
 	<origin rpy="0 0 0" xyz="0 0 0" />
@@ -402,9 +413,9 @@
     <parent link="frame"/>
     <child link="roller13"/>
-<xacro:if value="$(arg gazebo)">
-    <dynamics damping="10.0" friction="5.0"/>
-</xacro:if>
-   </joint>
-   <link name="roller13" type="fixed" > <!-- Every roller is 0.1 from previous center -->
+   <xacro:if value="$(arg gazebo)">
+    <dynamics damping="10.0" friction="5.0"/>
+   </xacro:if>
+   </joint>
+   <link name="roller13" type="fixed" >
        <visual>
 	<origin rpy="0 0 0" xyz="0 0 0" />
@@ -431,9 +442,9 @@
     <parent link="frame"/>
     <child link="roller14"/>
-<xacro:if value="$(arg gazebo)">
-    <dynamics damping="10.0" friction="5.0"/>
-</xacro:if>
-   </joint>
-   <link name="roller14" type="fixed" > <!-- Every roller is 0.1 from previous center -->
+   <xacro:if value="$(arg gazebo)">
+    <dynamics damping="10.0" friction="5.0"/>
+   </xacro:if>
+   </joint>
+   <link name="roller14" type="fixed" >
        <visual>
 	<origin rpy="0 0 0" xyz="0 0 0" />
@@ -460,9 +471,9 @@
     <parent link="frame"/>
     <child link="roller15"/>
-<xacro:if value="$(arg gazebo)">
-    <dynamics damping="10.0" friction="5.0"/>
-</xacro:if>
-   </joint>
-   <link name="roller15" type="fixed" > <!-- Every roller is 0.1 from previous center -->
+   <xacro:if value="$(arg gazebo)">
+    <dynamics damping="10.0" friction="5.0"/>
+   </xacro:if>
+   </joint>
+   <link name="roller15" type="fixed" >
        <visual>
 	<origin rpy="0 0 0" xyz="0 0 0" />
@@ -489,36 +500,35 @@
     <parent link="frame"/>
     <child link="roller16"/>
-<xacro:if value="$(arg gazebo)">
-    <dynamics damping="10.0" friction="5.0"/>
+   <xacro:if value="$(arg gazebo)">
+    <dynamics damping="10.0" friction="5.0"/>
+   </xacro:if>
+   </joint>
+   <link name="roller16" type="fixed" >
+       <visual>
+	<origin rpy="0 0 0" xyz="0 0 0" />
+  	  <geometry>
+		<mesh filename="package://sawyer_irl_project/meshes/roller.stl"/>
+	  </geometry>
+       </visual>
+	<collision>
+          <origin rpy="1.5708 0 0" xyz="0 0 0" />
+  	  <geometry>
+		<cylinder length="0.26" radius="0.04"/>
+	  </geometry>
+	</collision>
+    <inertial>
+       <origin rpy="0 0 0" xyz="0 0 0"/>
+       <mass value="11.56"/>
+      <inertia ixx="0.01" ixy="0" ixz="0" iyy="0.09" iyz="0" izz="0.09"/>
+    </inertial>
+    </link>
 </xacro:if>
-   </joint>
-   <link name="roller16" type="fixed" > <!-- Every roller is 0.1 from previous center -->
-       <visual>
-	<origin rpy="0 0 0" xyz="0 0 0" />
-  	  <geometry>
-		<mesh filename="package://sawyer_irl_project/meshes/roller.stl"/>
-	  </geometry>
-       </visual>
-	<collision>
-          <origin rpy="1.5708 0 0" xyz="0 0 0" />
-  	  <geometry>
-		<cylinder length="0.26" radius="0.04"/>
-	  </geometry>
-	</collision>
-    <inertial>
-       <origin rpy="0 0 0" xyz="0 0 0"/>
-       <mass value="11.56"/>
-      <inertia ixx="0.01" ixy="0" ixz="0" iyy="0.09" iyz="0" izz="0.09"/>
-    </inertial>
-    </link>
   <joint name="frame_to_belt" type="fixed">
     <origin rpy="0 0 0" xyz="0.75 0 0.73" />
-    <!--axis xyz="1 0 0" />
-    <limit lower="0.0" upper="6.28319" effort="1000.0" velocity="0.5"/-->
     <parent link="frame"/>
     <child link="belt"/>
-<xacro:if value="$(arg gazebo)">
-    <dynamics damping="10.0" friction="5.0"/>
-</xacro:if>
+   <xacro:if value="$(arg gazebo)">
+    <dynamics damping="10.0" friction="5.0"/>
+   </xacro:if>
    </joint>
    <link name="belt" type="fixed" >
@@ -541,5 +551,72 @@
     </inertial>
     </link>
-   <!--transmission name="tran1">
+<xacro:if value="$(arg load_railings)">
+<!-- The reason why these are initialized w.r.t the world frame is because
+we want floating joints above the conveyor and w.r.t the frame will not do that -->
+  <joint name="frame_railing1_joint" type="fixed" >
+        <origin xyz="0.6 0.0 0.82" rpy="0.0 0.0 0.0"/>
+        <parent link="world" />
+        <child link="railing1"/>
+  </joint>
+  <joint name="frame_railing2_joint" type="fixed" >
+        <origin xyz="0.9 0.0 0.82" rpy="0.0 0.0 0.0"/>
+        <parent link="world" />
+        <child link="railing2"/>
+  </joint>
+<link name="railing1">
+    <collision>
+      <origin xyz="0 0 0.0" rpy="0 0 0"/>
+      <geometry>
+        <box size="0.01 1.5 0.01"/>-
+      </geometry>
+    </collision>
+    <visual>
+      <origin xyz="0 0 0.0" rpy="0 0 0"/>
+      <geometry>
+        <box size="0.01 1.5 0.01"/>-
+      </geometry>
+    </visual>
+    <inertial>
+      <origin xyz="0 0 0.0" rpy="0 0 0"/>
+      <mass value="1"/>
+      <inertia
+        ixx="1" ixy="0.0" ixz="0.0"
+        iyy="1" iyz="0.0"
+        izz="1"/>
+    </inertial>
+  </link>
+  <gazebo reference="railing1">
+      <mu1>0.0000001</mu1>
+      <mu2>0.0000001</mu2>
+  </gazebo>
+  <link name="railing2">
+    <collision>
+      <origin xyz="0 0 0.0" rpy="0 0 0"/>
+      <geometry>
+        <box size="0.01 1.5 0.01"/>-
+      </geometry>
+    </collision>
+    <visual>
+      <origin xyz="0 0 0.0" rpy="0 0 0"/>
+      <geometry>
+        <box size="0.01 1.5 0.01"/>-
+      </geometry>
+    </visual>
+    <inertial>
+      <origin xyz="0 0 0.0" rpy="0 0 0"/>
+      <mass value="1"/>
+      <inertia
+        ixx="1" ixy="0.0" ixz="0.0"
+        iyy="1" iyz="0.0"
+        izz="1"/>
+    </inertial>
+  </link>
+  <gazebo reference="railing2">
+      <mu1>0.0000001</mu1>
+      <mu2>0.0000001</mu2>
+  </gazebo>
+</xacro:if>
+<xacro:if value="$(arg load_motors)">
+   <transmission name="tran1">
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
File: urdf/sawyer_combined.urdf.xacro (robot description, xacro)
@@ -1,3 +1,5 @@
 <?xml version="1.0" ?>
+<!-- Author: Prasanth Suresh (ps32611@uga.edu); Description: Sawyer Robot combined with Robotiq Gripper URDF -->
+<!-- Do not edit/replicate without permission -->
 <robot name="sawyer" xmlns:xacro="http://www.ros.org/wiki/xacro">
   <xacro:arg name="gazebo" default="true"/>
@@ -11,31 +13,61 @@
     <xacro:arg name="electric_gripper" value="${electric_gripper}"/>
   </xacro:include>
+  <link name="world"/>
+<!-- Use a cylinder in place of the actual gripper. Used for testing and tuning -->
+<xacro:arg name="use_cylinder_end" default="false"/>
+<xacro:if value="$(arg use_cylinder_end)">
+  <joint name="right_gripper_base_joint" type="fixed" >
+        <origin xyz="0.0 0.0 0.1" rpy="0.0 0.0 1.5707"/>
+        <parent link="right_hand" />
+        <child link="cylinder_end" />
+    </joint>
+  <link name="cylinder_end">
+    <collision>
+      <origin xyz="0 0 0.0" rpy="0 0 0"/>
+      <geometry>
+        <cylinder length="0.15" radius="0.061"/>
+      </geometry>
+    </collision>
+    <visual>
+      <origin xyz="0 0 0.0" rpy="0 0 0"/>
+      <geometry>
+        <cylinder length="0.15" radius="0.061"/>
+      </geometry>
+    </visual>
+    <inertial>
+      <origin xyz="0 0 0" rpy="0 0 0"/>
+      <mass value="2.5"/>
+      <inertia ixx="0.007013" ixy="0" ixz="0" iyy="0.007013" iyz="0" izz="0.004651"/>
+    </inertial>
+  </link>
+</xacro:if>
+<xacro:arg name="robotiqgripper" default="false"/>
+<xacro:if value="$(arg robotiqgripper)">
   <xacro:include filename="$(find robotiq_2f_85_gripper_visualization)/urdf/robotiq_arg2f_85_model.xacro">
   </xacro:include>
-  <link name="world"/>
   <joint name="right_gripper_base_joint" type="fixed" >
-        <origin xyz="0.0 0.0 0.001" rpy="0.0 0.0 1.5707"/>
-        <parent link="right_hand" />
-        <child link="right_gripper_base" />
-    </joint>
-    <link name="right_gripper_base"/>
-    <joint name="robotiq_c_model_adapter" type="fixed" >
-        <origin xyz="0.0 0.0 0.00" rpy="0.0 0.0 0.0"/>
-        <parent link="right_gripper_base" />
-        <child link="robotiq_arg2f_base_link" />
-    </joint>
-    <joint name="right_gripper_tip_joint" type="fixed">
-      <origin rpy="0 0 0" xyz="0 0 0.1268"/>
-      <parent link="robotiq_arg2f_base_link"/>
-      <child link="right_gripper_tip"/>
-    </joint>
-    <!-- Electric Gripper Tip link -->
-    <link name="right_gripper_tip">
-      <inertial>
-        <origin xyz="0 0 0" rpy="0 0 0"/>
-        <mass value="2e-06"/>
-        <inertia ixx="1.1e-09" ixy="0" ixz="0" iyy="1.1e-09" iyz="0" izz="1.1e-09"/>
-      </inertial>
-    </link>
+    <origin xyz="0.0 0.0 0.001" rpy="0.0 0.0 1.5707"/>
+    <parent link="right_hand" />
+    <child link="right_gripper_base" />
+  </joint>
+  <link name="right_gripper_base"/>
+  <joint name="robotiq_c_model_adapter" type="fixed" >
+    <origin xyz="0.0 0.0 0.00" rpy="0.0 0.0 0.0"/>
+    <parent link="right_gripper_base" />
+    <child link="robotiq_arg2f_base_link" />
+  </joint>
+  <joint name="right_gripper_tip_joint" type="fixed">
+    <origin rpy="0 0 0" xyz="0 0 0.1268"/>
+    <parent link="robotiq_arg2f_base_link"/>
+    <child link="right_gripper_tip"/>
+  </joint>
+  <link name="right_gripper_tip">
+    <inertial>
+      <origin xyz="0 0 0" rpy="0 0 0"/>
+      <mass value="2e-06"/>
+      <inertia ixx="1.1e-09" ixy="0" ixz="0" iyy="1.1e-09" iyz="0" izz="1.1e-09"/>
+    </inertial>
+  </link>
+</xacro:if>
   <joint name="fixed" type="fixed">
       <parent link="world"/>

File: urdf/sawyer_lab.urdf.xacro (robot description, xacro)
@@ -1,4 +1,7 @@
 <?xml version="1.0"?>
+<!-- Author: Prasanth Suresh(ps32611@uga.edu); Description: Hardman Hall Rm 230 lab environment for Sawyer Robot -->
+<!-- Do not edit/replicate without permission -->
 <robot name="sawyer_lab" xmlns:xacro="http://www.ros.org/wiki/xacro">
+<!-- Currently not used -->
   <link name="world"/>
   <link name="lab">

Commit message: Merged two_scara_collaboration with this pkg

File: urdf/conveyor.urdf.xacro (robot description, xacro)
@@ -354,5 +354,5 @@
     <limit lower="0.0" upper="6.28319" effort="1000.0" velocity="0.5"/>
     <parent link="frame"/>
-    <child link="roller11"/>
+    <child link="roller11"/>SpawnModel: Failure - entity format is invalid.
    <xacro:if value="$(arg gazebo)">
     <dynamics damping="10.0" friction="5.0"/>
@@ -444,5 +444,5 @@
    <xacro:if value="$(arg gazebo)">
     <dynamics damping="10.0" friction="5.0"/>
-   </xacro:if>
+   </xacro:if>SpawnModel: Failure - entity format is invalid.
    </joint>
    <link name="roller14" type="fixed" >
