Commit message: Many changes

File: urdf/conveyor.urdf.xacro (robot description, xacro)
@@ -58,470 +58,4 @@
       </inertial>
     </link>
-<xacro:if value="$(arg load_rollers)">
-  <joint name="frame_to_roller1" type="revolute">
-    <origin xyz="0.75 -0.7 0.73" rpy="0 0 0"/>
-    <axis xyz="1 0 0" />
-    <limit lower="0.0" upper="6.28319" effort="1000.0" velocity="0.5"/>
-    <parent link="frame"/>
-    <child link="roller1"/>
-   <xacro:if value="$(arg gazebo)">
-    <dynamics damping="10.0" friction="5.0"/>
-   </xacro:if>
-   </joint>
-   <link name="roller1" type="fixed" >
-       <visual>
-	<origin rpy="0 0 0" xyz="0 0 0" />
-  	  <geometry>
-		<mesh filename="package://sawyer_irl_project/meshes/roller.stl"/>
-	  </geometry>
-       </visual>
-	<collision>
-          <origin rpy="1.5708 0 0" xyz="0 0 0" />
-  	  <geometry>
-		<cylinder length="0.26" radius="0.04"/>
-	  </geometry>
-	</collision>
-    <inertial>
-       <origin rpy="0 0 0" xyz="0 0 0"/>
-       <mass value="11.56"/>
-      <inertia ixx="0.01" ixy="0" ixz="0" iyy="0.09" iyz="0" izz="0.09"/>
-    </inertial>
-    </link>
-  <joint name="frame_to_roller2" type="revolute">
-    <origin rpy="0 0 0" xyz="0.75 -0.6 0.73" />
-    <axis xyz="1 0 0" />
-    <limit lower="0.0" upper="6.28319" effort="1000.0" velocity="0.5"/>
-    <parent link="frame"/>
-    <child link="roller2"/>
-   <xacro:if value="$(arg gazebo)">
-    <dynamics damping="10.0" friction="5.0"/>
-   </xacro:if>
-   </joint>
-   <link name="roller2" type="fixed" >
-       <visual>
-	<origin rpy="0 0 0" xyz="0 0 0" />
-  	  <geometry>
-		<mesh filename="package://sawyer_irl_project/meshes/roller.stl"/>
-	  </geometry>
-       </visual>
-	<collision>
-          <origin rpy="1.5708 0 0" xyz="0 0 0" />
-  	  <geometry>
-		<cylinder length="0.26" radius="0.04"/>
-	  </geometry>
-	</collision>
-    <inertial>
-       <origin rpy="0 0 0" xyz="0 0 0"/>
-       <mass value="11.56"/>
-      <inertia ixx="0.01" ixy="0" ixz="0" iyy="0.09" iyz="0" izz="0.09"/>
-    </inertial>
-    </link>
-   <joint name="frame_to_roller3" type="revolute">
-    <origin rpy="0 0 0" xyz="0.75 -0.5 0.73" />
-    <axis xyz="1 0 0" />
-    <limit lower="0.0" upper="6.28319" effort="1000.0" velocity="0.5"/>
-    <parent link="frame"/>
-    <child link="roller3"/>
-   <xacro:if value="$(arg gazebo)">
-    <dynamics damping="10.0" friction="5.0"/>
-   </xacro:if>
-   </joint>
-   <link name="roller3" type="fixed" >
-       <visual>
-	<origin rpy="0 0 0" xyz="0 0 0" />
-  	  <geometry>
-		<mesh filename="package://sawyer_irl_project/meshes/roller.stl"/>
-	  </geometry>
-       </visual>
-	<collision>
-          <origin rpy="1.5708 0 0" xyz="0 0 0" />
-  	  <geometry>
-		<cylinder length="0.26" radius="0.04"/>
-	  </geometry>
-	</collision>
-    <inertial>
-       <origin rpy="0 0 0" xyz="0 0 0"/>
-       <mass value="11.56"/>
-      <inertia ixx="0.01" ixy="0" ixz="0" iyy="0.09" iyz="0" izz="0.09"/>
-    </inertial>
-    </link>
-   <joint name="frame_to_roller4" type="revolute">
-    <origin rpy="0 0 0" xyz="0.75 -0.4 0.73" />
-    <axis xyz="1 0 0" />
-    <limit lower="0.0" upper="6.28319" effort="1000.0" velocity="0.5"/>
-    <parent link="frame"/>
-    <child link="roller4"/>
-   <xacro:if value="$(arg gazebo)">
-    <dynamics damping="10.0" friction="5.0"/>
-   </xacro:if>
-   </joint>
-   <link name="roller4" type="fixed" >
-       <visual>
-	<origin rpy="0 0 0" xyz="0 0 0" />
-  	  <geometry>
-		<mesh filename="package://sawyer_irl_project/meshes/roller.stl"/>
-	  </geometry>
-       </visual>
-	<collision>
-          <origin rpy="1.5708 0 0" xyz="0 0 0" />
-  	  <geometry>
-		<cylinder length="0.26" radius="0.04"/>
-	  </geometry>
-	</collision>
-    <inertial>
-       <origin rpy="0 0 0" xyz="0 0 0"/>
-       <mass value="11.56"/>
-      <inertia ixx="0.01" ixy="0" ixz="0" iyy="0.09" iyz="0" izz="0.09"/>
-    </inertial>
-    </link>
-   <joint name="frame_to_roller5" type="revolute">
-    <origin rpy="0 0 0" xyz="0.75 -0.3 0.73" />
-    <axis xyz="1 0 0" />
-    <limit lower="0.0" upper="6.28319" effort="1000.0" velocity="0.5"/>
-    <parent link="frame"/>
-    <child link="roller5"/>
-   <xacro:if value="$(arg gazebo)">
-    <dynamics damping="10.0" friction="5.0"/>
-   </xacro:if>
-   </joint>
-   <link name="roller5" type="fixed" >
-       <visual>
-	<origin rpy="0 0 0" xyz="0 0 0" />
-  	  <geometry>
-		<mesh filename="package://sawyer_irl_project/meshes/roller.stl"/>
-	  </geometry>
-       </visual>
-	<collision>
-          <origin rpy="1.5708 0 0" xyz="0 0 0" />
-  	  <geometry>
-		<cylinder length="0.26" radius="0.04"/>
-	  </geometry>
-	</collision>
-    <inertial>
-       <origin rpy="0 0 0" xyz="0 0 0"/>
-       <mass value="11.56"/>
-      <inertia ixx="0.01" ixy="0" ixz="0" iyy="0.09" iyz="0" izz="0.09"/>
-    </inertial>
-    </link>
-   <joint name="frame_to_roller6" type="revolute">
-    <origin rpy="0 0 0" xyz="0.75 -0.2 0.73" />
-    <axis xyz="1 0 0" />
-    <limit lower="0.0" upper="6.28319" effort="1000.0" velocity="0.5"/>
-    <parent link="frame"/>
-    <child link="roller6"/>
-   <xacro:if value="$(arg gazebo)">
-    <dynamics damping="10.0" friction="5.0"/>
-   </xacro:if>
-   </joint>
-   <link name="roller6" type="fixed" >
-       <visual>
-	<origin rpy="0 0 0" xyz="0 0 0" />
-  	  <geometry>
-		<mesh filename="package://sawyer_irl_project/meshes/roller.stl"/>
-	  </geometry>
-       </visual>
-	<collision>
-          <origin rpy="1.5708 0 0" xyz="0 0 0" />
-  	  <geometry>
-		<cylinder length="0.26" radius="0.04"/>
-	  </geometry>
-	</collision>
-    <inertial>
-       <origin rpy="0 0 0" xyz="0 0 0"/>
-       <mass value="11.56"/>
-      <inertia ixx="0.01" ixy="0" ixz="0" iyy="0.09" iyz="0" izz="0.09"/>
-    </inertial>
-    </link>
-   <joint name="frame_to_roller7" type="revolute">
-    <origin rpy="0 0 0" xyz="0.75 -0.1 0.73" />
-    <axis xyz="1 0 0" />
-    <limit lower="0.0" upper="6.28319" effort="1000.0" velocity="0.5"/>
-    <parent link="frame"/>
-    <child link="roller7"/>
-   <xacro:if value="$(arg gazebo)">
-    <dynamics damping="10.0" friction="5.0"/>
-   </xacro:if>
-   </joint>
-   <link name="roller7" type="fixed" >
-       <visual>
-	<origin rpy="0 0 0" xyz="0 0 0" />
-  	  <geometry>
-		<mesh filename="package://sawyer_irl_project/meshes/roller.stl"/>
-	  </geometry>
-       </visual>
-	<collision>
-          <origin rpy="1.5708 0 0" xyz="0 0 0" />
-  	  <geometry>
-		<cylinder length="0.26" radius="0.04"/>
-	  </geometry>
-	</collision>
-    <inertial>
-       <origin rpy="0 0 0" xyz="0 0 0"/>
-       <mass value="11.56"/>
-      <inertia ixx="0.01" ixy="0" ixz="0" iyy="0.09" iyz="0" izz="0.09"/>
-    </inertial>
-    </link>
-   <joint name="frame_to_roller8" type="revolute">
-    <origin rpy="0 0 0" xyz="0.75 0 0.73" />
-    <axis xyz="1 0 0" />
-    <limit lower="0.0" upper="6.28319" effort="1000.0" velocity="0.5"/>
-    <parent link="frame"/>
-    <child link="roller8"/>
-   <xacro:if value="$(arg gazebo)">
-    <dynamics damping="10.0" friction="5.0"/>
-   </xacro:if>
-   </joint>
-   <link name="roller8" type="fixed" >
-       <visual>
-	<origin rpy="0 0 0" xyz="0 0 0" />
-  	  <geometry>
-		<mesh filename="package://sawyer_irl_project/meshes/roller.stl"/>
-	  </geometry>
-       </visual>
-	<collision>
-          <origin rpy="1.5708 0 0" xyz="0 0 0" />
-  	  <geometry>
-		<cylinder length="0.26" radius="0.04"/>
-	  </geometry>
-	</collision>
-    <inertial>
-       <origin rpy="0 0 0" xyz="0 0 0"/>
-       <mass value="11.56"/>
-      <inertia ixx="0.01" ixy="0" ixz="0" iyy="0.09" iyz="0" izz="0.09"/>
-    </inertial>
-    </link>
-   <joint name="frame_to_roller9" type="revolute">
-    <origin rpy="0 0 0" xyz="0.75 0.1 0.73" />
-    <axis xyz="1 0 0" />
-    <limit lower="0.0" upper="6.28319" effort="1000.0" velocity="0.5"/>
-    <parent link="frame"/>
-    <child link="roller9"/>
-   <xacro:if value="$(arg gazebo)">
-    <dynamics damping="10.0" friction="5.0"/>
-   </xacro:if>
-   </joint>
-   <link name="roller9" type="fixed" >
-       <visual>
-	<origin rpy="0 0 0" xyz="0 0 0" />
-  	  <geometry>
-		<mesh filename="package://sawyer_irl_project/meshes/roller.stl"/>
-	  </geometry>
-       </visual>
-	<collision>
-          <origin rpy="1.5708 0 0" xyz="0 0 0" />
-  	  <geometry>
-		<cylinder length="0.26" radius="0.04"/>
-	  </geometry>
-	</collision>
-    <inertial>
-       <origin rpy="0 0 0" xyz="0 0 0"/>
-       <mass value="11.56"/>
-      <inertia ixx="0.01" ixy="0" ixz="0" iyy="0.09" iyz="0" izz="0.09"/>
-    </inertial>
-    </link>
-   <joint name="frame_to_roller10" type="revolute">
-    <origin rpy="0 0 0" xyz="0.75 0.2 0.73" />
-    <axis xyz="1 0 0" />
-    <limit lower="0.0" upper="6.28319" effort="1000.0" velocity="0.5"/>
-    <parent link="frame"/>
-    <child link="roller10"/>
-   <xacro:if value="$(arg gazebo)">
-    <dynamics damping="10.0" friction="5.0"/>
-   </xacro:if>
-   </joint>
-   <link name="roller10" type="fixed" >
-       <visual>
-	<origin rpy="0 0 0" xyz="0 0 0" />
-  	  <geometry>
-		<mesh filename="package://sawyer_irl_project/meshes/roller.stl"/>
-	  </geometry>
-       </visual>
-	<collision>
-          <origin rpy="1.5708 0 0" xyz="0 0 0" />
-  	  <geometry>
-		<cylinder length="0.26" radius="0.04"/>
-	  </geometry>
-	</collision>
-    <inertial>
-       <origin rpy="0 0 0" xyz="0 0 0"/>
-       <mass value="11.56"/>
-      <inertia ixx="0.01" ixy="0" ixz="0" iyy="0.09" iyz="0" izz="0.09"/>
-    </inertial>
-    </link>
-   <joint name="frame_to_roller11" type="revolute">
-    <origin rpy="0 0 0" xyz="0.75 0.3 0.73" />
-    <axis xyz="1 0 0" />
-    <limit lower="0.0" upper="6.28319" effort="1000.0" velocity="0.5"/>
-    <parent link="frame"/>
-    <child link="roller11"/>SpawnModel: Failure - entity format is invalid.
-   <xacro:if value="$(arg gazebo)">
-    <dynamics damping="10.0" friction="5.0"/>
-   </xacro:if>
-   </joint>
-   <link name="roller11" type="fixed" >
-       <visual>
-	<origin rpy="0 0 0" xyz="0 0 0" />
-  	  <geometry>
-		<mesh filename="package://sawyer_irl_project/meshes/roller.stl"/>
-	  </geometry>
-       </visual>
-	<collision>
-          <origin rpy="1.5708 0 0" xyz="0 0 0" />
-  	  <geometry>
-		<cylinder length="0.26" radius="0.04"/>
-	  </geometry>
-	</collision>
-    <inertial>
-       <origin rpy="0 0 0" xyz="0 0 0"/>
-       <mass value="11.56"/>
-      <inertia ixx="0.01" ixy="0" ixz="0" iyy="0.09" iyz="0" izz="0.09"/>
-    </inertial>
-    </link>
-   <joint name="frame_to_roller12" type="revolute">
-    <origin rpy="0 0 0" xyz="0.75 0.3 0.73" />
-    <axis xyz="1 0 0" />
-    <limit lower="0.0" upper="6.28319" effort="1000.0" velocity="0.5"/>
-    <parent link="frame"/>
-    <child link="roller12"/>
-   <xacro:if value="$(arg gazebo)">
-    <dynamics damping="10.0" friction="5.0"/>
-   </xacro:if>
-   </joint>
-   <link name="roller12" type="fixed" >
-       <visual>
-	<origin rpy="0 0 0" xyz="0 0 0" />
-  	  <geometry>
-		<mesh filename="package://sawyer_irl_project/meshes/roller.stl"/>
-	  </geometry>
-       </visual>
-	<collision>
-          <origin rpy="1.5708 0 0" xyz="0 0 0" />
-  	  <geometry>
-		<cylinder length="0.26" radius="0.04"/>
-	  </geometry>
-	</collision>
-    <inertial>
-       <origin rpy="0 0 0" xyz="0 0 0"/>
-       <mass value="11.56"/>
-      <inertia ixx="0.01" ixy="0" ixz="0" iyy="0.09" iyz="0" izz="0.09"/>
-    </inertial>
-    </link>
-   <joint name="frame_to_roller13" type="revolute">
-    <origin rpy="0 0 0" xyz="0.75 0.4 0.73" />
-    <axis xyz="1 0 0" />
-    <limit lower="0.0" upper="6.28319" effort="1000.0" velocity="0.5"/>
-    <parent link="frame"/>
-    <child link="roller13"/>
-   <xacro:if value="$(arg gazebo)">
-    <dynamics damping="10.0" friction="5.0"/>
-   </xacro:if>
-   </joint>
-   <link name="roller13" type="fixed" >
-       <visual>
-	<origin rpy="0 0 0" xyz="0 0 0" />
-  	  <geometry>
-		<mesh filename="package://sawyer_irl_project/meshes/roller.stl"/>
-	  </geometry>
-       </visual>
-	<collision>
-          <origin rpy="1.5708 0 0" xyz="0 0 0" />
-  	  <geometry>
-		<cylinder length="0.26" radius="0.04"/>
-	  </geometry>
-	</collision>
-    <inertial>
-       <origin rpy="0 0 0" xyz="0 0 0"/>
-       <mass value="11.56"/>
-      <inertia ixx="0.01" ixy="0" ixz="0" iyy="0.09" iyz="0" izz="0.09"/>
-    </inertial>
-    </link>
-   <joint name="frame_to_roller14" type="revolute">
-    <origin rpy="0 0 0" xyz="0.75 0.5 0.73" />
-    <axis xyz="1 0 0" />
-    <limit lower="0.0" upper="6.28319" effort="1000.0" velocity="0.5"/>
-    <parent link="frame"/>
-    <child link="roller14"/>
-   <xacro:if value="$(arg gazebo)">
-    <dynamics damping="10.0" friction="5.0"/>
-   </xacro:if>SpawnModel: Failure - entity format is invalid.
-   </joint>
-   <link name="roller14" type="fixed" >
-       <visual>
-	<origin rpy="0 0 0" xyz="0 0 0" />
-  	  <geometry>
-		<mesh filename="package://sawyer_irl_project/meshes/roller.stl"/>
-	  </geometry>
-       </visual>
-	<collision>
-          <origin rpy="1.5708 0 0" xyz="0 0 0" />
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
File: urdf/onion_bin.urdf.xacro (robot description, xacro)
@@ -33,5 +33,6 @@
     </inertial>
   </link>
-  <!-- Box height is 0.7 m. top center of box w.r.t base of sawyer is at (0.1, 0.6, -0.2) in moveit -->
+  <!-- Box height is 0.7 m. top center of box w.r.t base of sawyer is at (0.1, 0.6, -0.2) in moveit.
+  So in order to get the box to floor height, move it down by -(0.2+0.7) -->
   <gazebo reference="onion_bin">
     <material>Gazebo/Green</material>

Commit message: first commit

File: urdf/conveyor.urdf.xacro (robot description, xacro)
@@ -90,9 +90,12 @@
   <joint name="frame_railing1_joint" type="fixed" >
         <origin xyz="0.6 0.0 0.82" rpy="0.0 0.0 0.0"/>
+        <!-- increased height for less onion hitting -->
+        <!-- <origin xyz="0.6 0.0 0.87" rpy="0.0 0.0 0.0"/> -->
         <parent link="world" />
         <child link="railing1"/>
   </joint>
   <joint name="frame_railing2_joint" type="fixed" >
-        <origin xyz="0.9 0.0 0.82" rpy="0.0 0.0 0.0"/>
+        <!-- <origin xyz="0.9 0.0 0.82" rpy="0.0 0.0 0.0"/> -->
+        <origin xyz="0.9 0.0 0.77" rpy="0.0 0.0 0.0"/>
         <parent link="world" />
         <child link="railing2"/>
@@ -790,5 +793,7 @@
     <gazebo reference="belt">
         <material>Gazebo/FlatBlack</material>
-        <mu1>0.0000001</mu1>
+        <!-- <mu1>0.0000001</mu1> -->
+        <!-- <mu1>0.5</mu1> -->
+        <mu1>5</mu1>
         <mu2>10.0</mu2>
     </gazebo>
